File: Starbie-My first PCB.kicad_pcb (KiCad board)
At the start: 2 copper layers, 84.8 x 84.6 mm, 12 parts, among them J1 Conn_01x04_Pin, J2 Conn_01x02_Pin, J3 Conn_01x08_Pin, Q1 Q_NPN_CBE, SW1 SW_Push, SW2 SW_Push, U1 XIAO-ESP32-C3-SMD, U2 DHT11

Commit message: fix drc errors
Routing:
- net GND: track 297.2 -> 272.1 mm
- net +3.3V: track 248.4 -> 231.8 mm
- net /SCL: track 138.3 -> 139.3 mm
Changed lines of the file:
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@@
 			(effects
 				(font
-					(size 0.635 0.635)
-					(thickness 0.1016)
+					(size 0.8 0.8)
+					(thickness 0.12)
 				)
 			)
@@
 			(effects
 				(font
-					(size 0.635 0.635)
-					(thickness 0.1016)
+					(size 0.8 0.8)
+					(thickness 0.12)
 				)
 			)
@@
 				(type solid)
 			)
-			(layer "F.SilkS")
+			(layer "F.Fab")
 		)
 		(fp_line
@@
 				(type solid)
 			)
-			(layer "F.SilkS")
+			(layer "F.Fab")
 		)
 		(fp_arc
@@
 	(gr_line
 		(start 109.921644 136.470487)
-		(end 109.921728 136.470486)
-		(stroke
-			(width 0.1)
-			(type default)
-		)
-		(layer "Edge.Cuts")
-	)
-	(gr_line
-		(start 109.921728 136.470486)
 		(end 109.123099 135.941635)
 		(stroke
@@
 	)
 	(gr_text "+3.3V"
-		(at 117.75 125.75 0)
+		(at 115.5 122 45)
 		(layer "B.SilkS")
 		(effects
@@
 	)
 	(gr_text "GND"
-		(at 159.5 75.25 0)
+		(at 160.5 76.5 0)
 		(layer "B.SilkS")
 		(effects
@@
 	)
 	(gr_text "GND"
-		(at 180.75 63 0)
+		(at 182 64.5 0)
 		(layer "B.SilkS")
 		(effects
@@
 	)
 	(segment
-		(start 136.5 78.5)
-		(end 134 76)
-		(width 0.2)
-		(layer "B.Cu")
-		(net "+3.3V")
-	)
-	(segment
 		(start 167.865448 71.634552)
 		(end 171 68.5)
@@
 	(segment
 		(start 126.625 77.125)
-		(end 114.815795 65.315795)
+		(end 122 72.5)
 		(width 0.2)
 		(layer "B.Cu")
@@
 	)
 	(segment
-		(start 153.96 73.5)
-		(end 153.96 73.275)
-		(width 0.2)
-		(layer "B.Cu")
-		(net "+3.3V")
-	)
-	(segment
 		(start 117.55 89.45)
 		(end 136.26 108.16)
@@
 	)
 	(segment
-		(start 133.9 73.5)
-		(end 134 73.5)
-		(width 0.2)
-		(layer "B.Cu")
-		(net "+3.3V")
-	)
-	(segment
 		(start 116.338891 84.322631)
 		(end 122.75 84.322631)
@@
 	)
 	(segment
-		(start 122.75 84.322631)
-		(end 123.077369 84.322631)
-		(width 0.2)
-		(layer "B.Cu")
-		(net "+3.3V")
-	)
-	(segment
 		(start 136.5 78.5)
 		(end 143.2575 71.7425)
@@
 	)
 	(segment
-		(start 153.96 73.275)
-		(end 155.4925 71.7425)
-		(width 0.2)
-		(layer "B.Cu")
-		(net "+3.3V")
-	)
-	(segment
 		(start 156.75 86.91098)
 		(end 156.75 103.611846)
@@
 	)
 	(segment
-		(start 136.725 112)
-		(end 135.425 110.7)
-		(width 0.2)
-		(layer "F.Cu")
-		(net "GND")
-	)
-	(segment
 		(start 154.102214 111.25)
 		(end 153.590214 111.762)
@@
 	)
 	(segment
-		(start 159.75 111.25)
-		(end 159 111.25)
-		(width 0.2)
-		(layer "F.Cu")
-		(net "GND")
-	)
-	(segment
 		(start 168.578213 117.078213)
 		(end 168.75 117.25)
@@
 	)
 	(segment
-		(start 158.316553 109.942899)
-		(end 156.259452 112)
-		(width 0.2)
-		(layer "F.Cu")
-		(net "GND")
-	)
-	(segment
 		(start 136.487 111.762)
 		(end 136.26 111.535)
@@
 	)
 	(segment
-		(start 156.259452 112)
-		(end 136.725 112)
-		(width 0.2)
-		(layer "F.Cu")
-		(net "GND")
-	)
-	(segment
 		(start 177.25 62.25)
 		(end 172.870699 62.25)
@@
 	)
 	(segment
-		(start 158.506412 112.348515)
-		(end 158.506412 112.175651)
-		(width 0.2)
-		(layer "F.Cu")
-		(net "/SDA")
-	)
-	(segment
 		(start 153.851 107.771664)
 		(end 153.851 101.81337)
@@
 	)
 	(segment
-		(start 168.5 122.342103)
-		(end 168.421439 122.342103)
-		(width 0.2)
-		(layer "F.Cu")
-		(net "/SDA")
-	)
-	(segment
 		(start 157.895659 114.064173)
 		(end 158.506412 114.064173)
@@
 	)
 	(embedded_fonts no)
+	(segment
+		(start 150.5 103.25)
+		(end 151.5 103.08)
+		(width 0.2)
+		(layer "F.Cu")
+		(net "/SCL")
+	)
 )

Commit message: fix buzzer circuit and schematic erc warnings
Parts:
- moved D1 10.2 mm to (122.0, 72.5), turned to 135 degrees
- moved BZ1 7.60 mm to (136.5, 78.5), turned to 180 degrees
Connections:
- BZ1 pad 1: Net-(BZ1-+) -> +3.3V
- BZ1 pad 2: +3.3V -> Net-(BZ1--)
- D1 pad 1: Net-(BZ1-+) -> +3.3V
- D1 pad 2: +3.3V -> Net-(BZ1--)
- Q1 pad 1: Net-(BZ1-+) -> Net-(BZ1--)
Routing:
- net Net-(BZ1--): track 0.00 -> 51.1 mm
- net Net-(BZ1-+): track 51.1 -> 0.00 mm
Changed lines of the file:
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@@
 	(footprint "Diode_THT:D_DO-35_SOD27_P10.16mm_Horizontal"
 		(layer "F.Cu")
-		(at 114.815795 65.315795 -45)
+		(at 122 72.5 135)
 		(descr "Diode, DO-35_SOD27 series, Axial, Horizontal, pin pitch=10.16mm, length*diameter=4*2mm^2, http://www.diodes.com/_files/packages/DO-35.pdf")
 		(tags "Diode DO-35_SOD27 series Axial Horizontal pin pitch 10.16mm  length 4mm diameter 2mm")
@@
 			(remove_unused_layers no)
 			(roundrect_rratio 0.15625)
-			(net "Net-(BZ1-+)")
+			(net "+3.3V")
 			(pinfunction "K_1")
 			(pintype "passive")
@@
 			(layers "*.Cu" "*.Mask")
 			(remove_unused_layers no)
-			(net "+3.3V")
+			(net "Net-(BZ1--)")
 			(pinfunction "A_2")
 			(pintype "passive")
@@
 			(layers "*.Cu" "*.Mask")
 			(remove_unused_layers no)
-			(net "Net-(BZ1-+)")
+			(net "Net-(BZ1--)")
 			(pinfunction "C_1")
 			(pintype "passive")
@@
 	(footprint "Buzzer_Beeper:Buzzer_12x9.5RM7.6"
 		(layer "F.Cu")
-		(at 128.9 78.5)
+		(at 136.5 78.5 180)
 		(descr "Generic Buzzer, D12mm height 9.5mm with RM7.6mm")
 		(tags "buzzer")
@@
 			(layers "*.Cu" "*.Mask")
 			(remove_unused_layers no)
-			(net "Net-(BZ1-+)")
+			(net "+3.3V")
 			(pinfunction "+_1")
 			(pintype "passive")
@@
 			(layers "*.Cu" "*.Mask")
 			(remove_unused_layers no)
-			(net "+3.3V")
+			(net "Net-(BZ1--)")
 			(pinfunction "-_2")
 			(pintype "passive")
@@
 		(width 0.2)
 		(layer "F.Cu")
-		(net "Net-(BZ1-+)")
+		(net "Net-(BZ1--)")
 	)
 	(segment
@@
 		(width 0.2)
 		(layer "F.Cu")
-		(net "Net-(BZ1-+)")
+		(net "Net-(BZ1--)")
 	)
 	(segment
@@
 		(width 0.2)
 		(layer "F.Cu")
-		(net "Net-(BZ1-+)")
+		(net "Net-(BZ1--)")
 	)
 	(segment
@@
 		(width 0.2)
 		(layer "F.Cu")
-		(net "Net-(BZ1-+)")
+		(net "Net-(BZ1--)")
 	)
 	(segment
@@
 		(width 0.2)
 		(layer "F.Cu")
-		(net "Net-(BZ1-+)")
+		(net "Net-(BZ1--)")
 	)
 	(segment
@@
 		(width 0.2)
 		(layer "B.Cu")
-		(net "Net-(BZ1-+)")
+		(net "Net-(BZ1--)")
 	)
 	(segment
@@
 		(width 0.2)
 		(layer "B.Cu")
-		(net "Net-(BZ1-+)")
+		(net "Net-(BZ1--)")
 	)
 	(segment
@@
 		(width 0.2)
 		(layer "B.Cu")
-		(net "Net-(BZ1-+)")
+		(net "Net-(BZ1--)")
 	)
 	(segment
@@
 		(width 0.2)
 		(layer "B.Cu")
-		(net "Net-(BZ1-+)")
+		(net "Net-(BZ1--)")
 	)
 	(segment
@@
 		(width 0.2)
 		(layer "B.Cu")
-		(net "Net-(BZ1-+)")
+		(net "Net-(BZ1--)")
 	)
 	(segment
@@
 		(width 0.2)
 		(layer "B.Cu")
-		(net "Net-(BZ1-+)")
+		(net "Net-(BZ1--)")
 	)
 	(segment
@@
 		(width 0.2)
 		(layer "B.Cu")
-		(net "Net-(BZ1-+)")
+		(net "Net-(BZ1--)")
 	)
 	(zone
@@
 	)
 	(zone
-		(net "Net-(BZ1-+)")
+		(net "Net-(BZ1--)")
 		(layer "F.Cu")
 		(hatch none 0.1)
@@
 	)
 	(zone
-		(net "Net-(BZ1-+)")
+		(net "Net-(BZ1--)")
 		(layer "F.Cu")
 		(hatch none 0.1)
@@
 	)
 	(zone
-		(net "Net-(BZ1-+)")
+		(net "Net-(BZ1--)")
 		(layer "B.Cu")
 		(hatch none 0.1)
@@
 	)
 	(zone
-		(net "Net-(BZ1-+)")
+		(net "Net-(BZ1--)")
 		(layer "B.Cu")
 		(hatch none 0.1)
